File: hardware/lora_daq_module/lora_daq_module.kicad_pcb (KiCad board)
At the start: 2 copper layers, 0 parts

Commit message: updated power schematic to include power switching IC for battery/usb power, minor changes to lora module schematic, added footprints to all component and began with the preliminary layout based on data sheet and application note reccomendations for each component.
Parts:
- added C1: 0.1uF, Capacitor_SMD:C_0603_1608Metric, F.Cu at (137.2, 120.0)
- added C10: 1u, Capacitor_SMD:C_0603_1608Metric, F.Cu at (146.7, 97.5)
- added C11: 10n, Capacitor_SMD:C_0603_1608Metric, F.Cu at (118.5, 109.0)
- added C12: .1u, Capacitor_SMD:C_0603_1608Metric, F.Cu at (156.6, 118.2)
- added C13: 10n, Capacitor_SMD:C_0603_1608Metric, B.Cu at (162.7, 96.0)
- added C14: .47u, Capacitor_SMD:C_0603_1608Metric, F.Cu at (127.0, 95.9)
- added C15: 1u, Capacitor_SMD:C_0603_1608Metric, F.Cu at (144.7, 89.3)
- added C16: 1u, Capacitor_SMD:C_0603_1608Metric, F.Cu at (136.3, 99.4)
- added C17: 1u, Capacitor_SMD:C_0603_1608Metric, F.Cu at (140.9, 99.4)
- added C18: 10uF, Capacitor_SMD:C_1206_3216Metric, F.Cu at (131.7, 87.7)
- added C19: 33uF, Capacitor_SMD:C_1210_3225Metric, F.Cu at (132.7, 95.2)
- added C2: 47nF, Capacitor_SMD:C_0603_1608Metric, F.Cu at (126.2, 114.3)
- added C20: 1uF, Capacitor_SMD:C_0603_1608Metric, F.Cu at (117.9, 96.5)
- added C21: 1uF, Capacitor_SMD:C_0603_1608Metric, F.Cu at (117.9, 91.7)
- added C3: 0, Capacitor_SMD:C_0603_1608Metric, F.Cu at (168.7, 102.5)
- added C4: 0, Capacitor_SMD:C_0603_1608Metric, F.Cu at (166.4, 102.5)
- added C5: 1u, Capacitor_SMD:C_0603_1608Metric, F.Cu at (129.7, 107.2)
- added C6: .1u, Capacitor_SMD:C_0603_1608Metric, F.Cu at (128.2, 107.2)
- added C7: .1u, Capacitor_SMD:C_0603_1608Metric, F.Cu at (126.5, 107.2)
- added C8: 4.7u, Capacitor_SMD:C_1206_3216Metric, F.Cu at (124.5, 107.4)
- added C9: .1u, Capacitor_SMD:C_0603_1608Metric, F.Cu at (146.7, 96.0)
- added D3: SP0503BAHT, Package_TO_SOT_SMD:SOT-143, F.Cu at (126.0, 101.7)
- added D4: ~, LED_SMD:LED_0603_1608Metric, F.Cu at (125.2, 93.5)
- added D5: ~, LED_SMD:LED_0603_1608Metric, F.Cu at (115.7, 97.2)
- added D6: ~, LED_SMD:LED_0603_1608Metric, F.Cu at (113.7, 97.2)
- added D7: BAS40-04, Package_TO_SOT_SMD:SOT-23, F.Cu at (131.7, 116.0)
- added J1: JST3pinfemale, Connector_JST:JST_EH_B3B-EH-A_1x03_P2.50mm_Vertical, F.Cu at (121.4, 118.3)
- added J2: SMA_Edge_50Ω, Connector_Coaxial:SMA_Molex_73251-1153_EdgeMount_Horizontal, F.Cu at (173.1, 105.7)
- added J3: USB_C_Receptacle_USB2.0_14P, Connector_USB:USB_C_Receptacle_Molex_105450-0101, F.Cu at (112.1, 104.5)
- added J4: EXT_UART, Connector_JST:JST_EH_B3B-EH-A_1x03_P2.50mm_Vertical, F.Cu at (169.2, 119.2)
- added J5: SWD, Connector_PinHeader_2.54mm:PinHeader_2x03_P2.54mm_Vertical, F.Cu at (154.0, 85.2)
- added J6: Micro_SD_Card_Det1, Connector_Card:microSD_HC_Molex_104031-0811, B.Cu at (171.2, 90.2)
- added J7: Conn_01x02, Connector_PinHeader_2.54mm:PinHeader_1x02_P2.54mm_Vertical, F.Cu at (110.4, 90.5)
- added L1: 0, Resistor_SMD:R_0603_1608Metric, F.Cu at (167.5, 105.2)
- added L2: 3.3uH, Inductor_SMD:L_Coilcraft_LPS3010, F.Cu at (135.8, 91.2)
- added R1: 47k, Resistor_SMD:R_0603_1608Metric, F.Cu at (123.9, 113.5)
- added R10: 680k, Resistor_SMD:R_0603_1608Metric, F.Cu at (128.5, 95.9)
- added R11: 470k, Resistor_SMD:R_0603_1608Metric, F.Cu at (128.5, 98.9)
- added R12: 4.7k, Resistor_SMD:R_0603_1608Metric, F.Cu at (133.6, 100.0)
- added R13: 470Ω, Resistor_SMD:R_0603_1608Metric, F.Cu at (114.2, 94.2)
- added R14: 470Ω, Resistor_SMD:R_0603_1608Metric, F.Cu at (115.7, 94.2)
- added R15: 470Ω, Resistor_SMD:R_0603_1608Metric, F.Cu at (124.2, 91.0)
- added R16: 1kΩ, Resistor_SMD:R_0603_1608Metric, F.Cu at (120.9, 89.3)
- added R17: 10k_therm, Resistor_SMD:R_0603_1608Metric, F.Cu at (123.2, 87.5)
- added R18: 150k, Resistor_SMD:R_0603_1608Metric, F.Cu at (123.2, 89.0)
- added R19: 1kΩ, Resistor_SMD:R_0603_1608Metric, F.Cu at (123.4, 93.4)
- added R2: 220k, Resistor_SMD:R_0603_1608Metric, F.Cu at (129.2, 114.3)
- added R3: 1k, Resistor_SMD:R_0603_1608Metric, F.Cu at (127.7, 114.3)
- added R4: 5.1k, Resistor_SMD:R_0603_1608Metric, F.Cu at (121.6, 102.0)
- added R5: 5.1k, Resistor_SMD:R_0603_1608Metric, F.Cu at (121.6, 106.0)
- added R6: 4.7k, Resistor_SMD:R_0603_1608Metric, F.Cu at (164.9, 98.0)
- added R7: 4.7k, Resistor_SMD:R_0603_1608Metric, F.Cu at (146.7, 104.0)
- added R8: 4.7k, Resistor_SMD:R_0603_1608Metric, F.Cu at (146.7, 102.5)
- added R9: 4.7k, Resistor_SMD:R_0603_1608Metric, F.Cu at (154.7, 92.2)
- added TP1: cp2102_3v3reg, TestPoint:TestPoint_Pad_3.0x3.0mm, F.Cu at (109.9, 112.5)
- added U1: OPA333, Package_SO:SOIC-8_3.9x4.9mm_P1.27mm, F.Cu at (136.4, 112.1)
- added U2: ADS1115IDGS, Package_SO:TSSOP-10_3x3mm_P0.5mm, F.Cu at (137.2, 117.2)
- added U3: CP2102N-Axx-xQFN20, Package_DFN_QFN:SiliconLabs_QFN-20-1EP_3x3mm_P0.5mm_EP1.8x1.8mm, F.Cu at (130.2, 103.5)
- added U4: Wio-E5_STM32WLE5JC, LoRa-E5:LoRa-E5, F.Cu at (155.9, 101.5)
- added U5: CAT24C256, Package_SO:SOIC-8-1EP_3.9x4.9mm_P1.27mm_EP2.29x3mm, F.Cu at (156.7, 114.7)
- added U6: MCP1700x-330xxTT, Package_TO_SOT_SMD:SOT-23, F.Cu at (138.2, 97.2)
- added U7: TPS2116DRL, Package_TO_SOT_SMD:SOT-583-8, F.Cu at (130.8, 98.7)
- added U8: TPS63002, Package_SON:Texas_DRC0010J_ThermalVias, F.Cu at (131.8, 91.2)
- added U9: MCP73833, Package_SO:MSOP-10_3x3mm_P0.5mm, F.Cu at (120.7, 94.2)
Routing:
- net SCL: track 0.00 -> 33.5 mm, vias 0 -> 2
- net SDA: track 0.00 -> 33.0 mm, vias 0 -> 2
- net RX1: track 0.00 -> 32.7 mm, vias 0 -> 2
- net TX1: track 0.00 -> 31.6 mm, vias 0 -> 2
- net USB_RST: track 0.00 -> 23.7 mm, vias 0 -> 2
- net D-: track 0.00 -> 19.8 mm, vias 0 -> 2
- net D+: track 0.00 -> 15.1 mm
- net Net-(U1-+): track 0.00 -> 13.3 mm
- net VBUS: track 0.00 -> 8.80 mm, vias 0 -> 2
- net GND: track 0.00 -> 8.48 mm, vias 0 -> 7
- net +3.3V: track 0.00 -> 7.90 mm
- net Net-(J3-CC2): track 0.00 -> 7.07 mm, vias 0 -> 2
- net Net-(J3-CC1): track 0.00 -> 6.08 mm
- net Net-(U4-F5/~{RST}): track 0.00 -> 6.00 mm
- net /adc/sig0+: track 0.00 -> 5.54 mm
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- added copper zone on B.Cu, net GND
- added copper zone on F.Cu, net GND
- added copper zone on In1.Cu, net GND
- added copper zone on In2.Cu, net GND
Other:
- board outline added: 70 x 40 mm
- copper layers 2 -> 4
